File: PCB_Expert_in_Teams/pcb/AI_deputy_PCB/Haptic_Driver_Module.kicad_sch (KiCad schematic)
At the start: 23 parts, among them IC1 DA7280-00FVC, IC2 DA7281-00FVC, IC3 DA7282-00FVC, J10 OUTPUT Haptic B (Neck R), J11 OUTPUT Haptic C (Back), J12 Haptic Power and GND, J7 JST CONN from MCU, J9 OUTPUT Haptic A (Neck L)

Commit message: updating repo from desktop
Other:
- company: (none) -> Area 42 & Albers-Online Psykologi
- title: (none) -> AI Deputy
Changed lines of the file:
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@@
 	(generator_version "9.0")
 	(paper "A4")
+	(title_block
+		(title "AI Deputy")
+		(date "2025-09-24")
+		(rev "v0.1")
+		(company "Area 42 & Albers-Online Psykologi")
+		(comment 1 "SDU")
+		(comment 2 "Expert In Teams Semester Project")
+	)
 	(junction
 		(at 132.08 71.12)

Commit message: 29/10/update
Parts:
- IC1, IC2: footprint QFN65P300X300X84-12N -> EXT_AI_DEPUTY_Library:QFN65P300X300X84-12N
Changed lines of the file:
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@@
 	(title_block
 		(title "AI Deputy")
-		(date "2025-09-24")
+		(date "2025-10-29")
 		(rev "v0.1")
 		(company "Area 42 & Albers-Online Psykologi")
@@
 			)
 		)
-		(property "Footprint" "QFN65P300X300X84-12N"
+		(property "Footprint" "EXT_AI_DEPUTY_Library:QFN65P300X300X84-12N"
 			(at 158.75 193.98 0)
 			(effects
@@
 			)
 		)
-		(property "Footprint" "QFN65P300X300X84-12N"
+		(property "Footprint" "EXT_AI_DEPUTY_Library:QFN65P300X300X84-12N"
 			(at 158.75 130.48 0)
 			(effects

Commit message: update pcb from desktop
Parts:
- IC3: footprint QFN65P300X300X84-12N -> EXT_AI_DEPUTY_Library:QFN65P300X300X84-12N
Changed lines of the file:
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@@
 			)
 		)
-		(property "Footprint" "QFN65P300X300X84-12N"
+		(property "Footprint" "EXT_AI_DEPUTY_Library:QFN65P300X300X84-12N"
 			(at 73.66 242.24 0)
 			(effects

Commit message: pcb updates from desktop with schematic fix
Parts:
- R1, R5, R6: value 4.7k -> 3.3k
Changed lines of the file:
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@@
 			)
 		)
-		(property "Value" "4.7k"
+		(property "Value" "3.3k"
 			(at 57.912 34.29 0)
 			(effects
@@
 			)
 		)
-		(property "Value" "4.7k"
+		(property "Value" "3.3k"
 			(at 65.278 34.29 0)
 			(effects
@@
 			)
 		)
-		(property "Value" "4.7k"
+		(property "Value" "3.3k"
 			(at 73.152 34.29 0)
 			(effects

Commit message: update after lab session with gustav saturday
Parts:
- removed J12: Haptic Power and GND, Connector_JST:JST_XH_S2B-XH-A_1x02_P2.50mm_Horizontal, symbol Connector:Conn_01x02_Socket
- removed J7: JST CONN from MCU, Connector_JST:JST_XH_S3B-XH-A_1x03_P2.50mm_Horizontal, symbol Connector:Conn_01x03_Socket
- removed R1, R5, R6: 3.3k, Resistor_SMD:R_0805_2012Metric_Pad1.20x1.40mm_HandSolder, symbol Device:R
