File: PCB_Expert_in_Teams/pcb/AI_deputy_PCB/UART.kicad_sch (KiCad schematic)
At the start: 8 parts, among them IC8 FT231XS-R

Commit message: update pcb from desktop
Parts:
- IC8: footprint SOP64P599X175-20N -> EXT_AI_DEPUTY_Library:SOP64P599X175-20N
Changed lines of the file:
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@@
 			)
 		)
-		(property "Footprint" "SOP64P599X175-20N"
+		(property "Footprint" "EXT_AI_DEPUTY_Library:SOP64P599X175-20N"
 			(at 161.29 155.88 0)
 			(effects

Commit message: update schematic from desktop
Parts:
- removed C43: 4.7u, symbol Device:C
- C44, C46: footprint (none) -> Capacitor_SMD:C_0805_2012Metric_Pad1.18x1.45mm_HandSolder
- R37, R38, R39, R40: footprint (none) -> Resistor_SMD:R_0805_2012Metric_Pad1.20x1.40mm_HandSolder
Changed lines of the file:
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@@
-	)
-	(junction
-		(at 129.54 40.64)
-		(diameter 0)
-		(color 0 0 0 0)
 	)
 	(junction
 		(at 125.73 87.63)
-		(diameter 0)
-		(color 0 0 0 0)
-	)
-	(junction
-		(at 129.54 48.26)
 		(diameter 0)
 		(color 0 0 0 0)
@@
 			)
 		)
-		(property "Footprint" ""
+		(property "Footprint" "Capacitor_SMD:C_0805_2012Metric_Pad1.18x1.45mm_HandSolder"
 			(at 126.6952 96.52 0)
 			(effects
@@
 	)
 	(symbol
-		(lib_id "Device:C")
-		(at 129.54 44.45 0)
-		(unit 1)
-		(exclude_from_sim no)
-		(in_bom yes)
-		(on_board yes)
-		(dnp no)
-		(property "Reference" "C43"
-			(at 121.666 43.18 0)
-			(effects
-				(font
-					(size 1.27 1.27)
-				)
-				(justify left)
-			)
-		)
-		(property "Value" "4.7u"
-			(at 121.666 45.72 0)
-			(effects
-				(font
-					(size 1.27 1.27)
-				)
-				(justify left)
-			)
-		)
-		(property "Footprint" ""
-			(at 130.5052 48.26 0)
-			(effects
-				(font
-					(size 1.27 1.27)
-				)
-				(hide yes)
-			)
-		)
-		(property "Datasheet" "~"
-			(at 129.54 44.45 0)
-			(effects
-				(font
-					(size 1.27 1.27)
-				)
-				(hide yes)
-			)
-		)
-		(property "Description" "Unpolarized capacitor"
-			(at 129.54 44.45 0)
-			(effects
-				(font
-					(size 1.27 1.27)
-				)
-				(hide yes)
-			)
-		)
-		(pin "2"
-		)
-		(pin "1"
-		)
-		(instances
-			(project ""
-				(path "/3784b751-4d5b-4452-8288-14e483e1cb48/87f65698-0461-47ba-97ee-9540500b8d33"
-					(reference "C43")
-					(unit 1)
-				)
-			)
-		)
-	)
-	(symbol
 		(lib_id "Device:R")
 		(at 170.18 95.25 180)
@@
 			)
 		)
-		(property "Footprint" ""
+		(property "Footprint" "Resistor_SMD:R_0805_2012Metric_Pad1.20x1.40mm_HandSolder"
 			(at 171.958 95.25 90)
 			(effects
@@
 			)
 		)
-		(property "Footprint" ""
+		(property "Footprint" "Resistor_SMD:R_0805_2012Metric_Pad1.20x1.40mm_HandSolder"
 			(at 123.19 80.518 90)
 			(effects
@@
 			)
 		)
-		(property "Footprint" ""
+		(property "Footprint" "Capacitor_SMD:C_0805_2012Metric_Pad1.18x1.45mm_HandSolder"
 			(at 141.9352 48.26 0)
 			(effects
@@
 			)
 		)
-		(property "Footprint" ""
+		(property "Footprint" "Resistor_SMD:R_0805_2012Metric_Pad1.20x1.40mm_HandSolder"
 			(at 123.19 77.978 90)
 			(effects
@@
 			)
 		)
-		(property "Footprint" ""
+		(property "Footprint" "Resistor_SMD:R_0805_2012Metric_Pad1.20x1.40mm_HandSolder"
 			(at 171.958 106.68 90)
 			(effects

Commit message: fixed small things, push from laptop
Parts:
- R37: value R -> 27
Connections:
- net +: now reaches IC8.11 (USBDP), R37.2
- net -: now reaches IC8.12 (USBDM), R38.2
Other:
- moved on the sheet: R37, R38
Changed lines of the file:
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@@
-	(wire
-		(pts
-			(xy 127 76.2) (xy 132.08 76.2)
-		)
-		(stroke
-			(width 0)
-			(type default)
-		)
-	)
 	(wire
 		(pts
@@
 	(wire
 		(pts
-			(xy 111.76 76.2) (xy 119.38 76.2)
+			(xy 111.76 76.2) (xy 113.03 76.2)
 		)
 		(stroke
@@
 	(wire
 		(pts
-			(xy 127 78.74) (xy 132.08 78.74)
-		)
-		(stroke
-			(width 0)
-			(type default)
-		)
-	)
-	(wire
-		(pts
 			(xy 129.54 71.12) (xy 129.54 67.31)
 		)
@@
 	(wire
 		(pts
-			(xy 111.76 78.74) (xy 119.38 78.74)
+			(xy 111.76 78.74) (xy 113.03 78.74)
 		)
 		(stroke
@@
 			(width 0)
 			(type default)
+		)
+	)
+	(global_label "-"
+		(shape input)
+		(at 132.08 76.2 180)
+		(fields_autoplaced yes)
+		(effects
+			(font
+				(size 1.27 1.27)
+			)
+			(justify right)
+		)
+		(property "Intersheetrefs" "${INTERSHEET_REFS}"
+			(at 127.5224 76.2 0)
+			(effects
+				(font
+					(size 1.27 1.27)
+				)
+				(justify right)
+				(hide yes)
+			)
+		)
+	)
+	(global_label "+"
+		(shape input)
+		(at 120.65 78.74 0)
+		(fields_autoplaced yes)
+		(effects
+			(font
+				(size 1.27 1.27)
+			)
+			(justify left)
+		)
+		(property "Intersheetrefs" "${INTERSHEET_REFS}"
+			(at 125.2076 78.74 0)
+			(effects
+				(font
+					(size 1.27 1.27)
+				)
+				(justify left)
+				(hide yes)
+			)
+		)
+	)
+	(global_label "-"
+		(shape input)
+		(at 120.65 76.2 0)
+		(fields_autoplaced yes)
+		(effects
+			(font
+				(size 1.27 1.27)
+			)
+			(justify left)
+		)
+		(property "Intersheetrefs" "${INTERSHEET_REFS}"
+			(at 125.2076 76.2 0)
+			(effects
+				(font
+					(size 1.27 1.27)
+				)
+				(justify left)
+				(hide yes)
+			)
 		)
 	)
@@
 				)
 				(justify left)
+				(hide yes)
+			)
+		)
+	)
+	(global_label "+"
+		(shape input)
+		(at 132.08 78.74 180)
+		(fields_autoplaced yes)
+		(effects
+			(font
+				(size 1.27 1.27)
+			)
+			(justify right)
+		)
+		(property "Intersheetrefs" "${INTERSHEET_REFS}"
+			(at 127.5224 78.74 0)
+			(effects
+				(font
+					(size 1.27 1.27)
+				)
+				(justify right)
 				(hide yes)
 			)
@@
 	(symbol
 		(lib_id "Device:R")
-		(at 123.19 78.74 90)
+		(at 116.84 78.74 90)
 		(unit 1)
 		(exclude_from_sim no)
@@
 		(dnp no)
 		(property "Reference" "R37"
-			(at 123.444 81.534 90)
-			(effects
-				(font
-					(size 1.27 1.27)
-				)
-			)
-		)
-		(property "Value" "R"
-			(at 123.444 84.074 90)
+			(at 117.094 81.534 90)
+			(effects
+				(font
+					(size 1.27 1.27)
+				)
+			)
+		)
+		(property "Value" "27"
+			(at 117.094 84.074 90)
 			(effects
 				(font
@@
 		)
 		(property "Footprint" "Resistor_SMD:R_0805_2012Metric_Pad1.20x1.40mm_HandSolder"
-			(at 123.19 80.518 90)
+			(at 116.84 80.518 90)
 			(effects
 				(font
@@
 		)
 		(property "Datasheet" "~"
-			(at 123.19 78.74 0)
+			(at 116.84 78.74 0)
 			(effects
 				(font
@@
 		)
 		(property "Description" "Resistor"
-			(at 123.19 78.74 0)
+			(at 116.84 78.74 0)
 			(effects
 				(font
@@
 	(symbol
 		(lib_id "Device:R")
-		(at 123.19 76.2 90)
+		(at 116.84 76.2 90)
 		(unit 1)
 		(exclude_from_sim no)
@@
 		(dnp no)
 		(property "Reference" "R38"
-			(at 123.444 71.374 90)
+			(at 117.094 71.374 90)
 			(effects
 				(font
@@
 		)
 		(property "Value" "27"
-			(at 123.444 73.914 90)
+			(at 117.094 73.914 90)
 			(effects
 				(font
@@
 		)
 		(property "Footprint" "Resistor_SMD:R_0805_2012Metric_Pad1.20x1.40mm_HandSolder"
-			(at 123.19 77.978 90)
+			(at 116.84 77.978 90)
 			(effects
 				(font
@@
 		)
 		(property "Datasheet" "~"
-			(at 123.19 76.2 0)
+			(at 116.84 76.2 0)
 			(effects
 				(font
@@
 		)
 		(property "Description" "Resistor"
-			(at 123.19 76.2 0)
-			(effects
-				(font
+			(at 116.84 76.2 0)
+			(effects
+				(font

Commit message: finished PCB design and gerbers are in directory
Parts:
- removed R39, R40: 100k, Resistor_SMD:R_0805_2012Metric_Pad1.20x1.40mm_HandSolder, symbol Device:R
- added C62: 100n, Capacitor_SMD:C_0805_2012Metric_Pad1.18x1.45mm_HandSolder, symbol Device:C
- added R6: 10k, Resistor_SMD:R_0805_2012Metric_Pad1.20x1.40mm_HandSolder, symbol Device:R
- C46: value 100n -> 1u
Connections:
- net +3V3: now also C46.1, IC8.13 (3V3OUT), R6.1
- net GND: now also C62.2
- new net: C62.1, IC8.14 (RESET#), R6.2
- no-connect marks 9 -> 10
