File: PCB_Expert_in_Teams/pcb/AI_deputy_PCB/AI_deputy_PCB.kicad_sch (KiCad schematic)
At the start: 28 parts, among them J1 Piezo Electric, J15 Conn_01x04_Socket, J3 Haptic Power and GND, J4 UART, J5 JST CONN from MCU, J6 JTAG, Q1 NMOS IRLZ44NPBF, U2 ESP32-WROOM-32UE

Commit message: extra commit to make sure i get everythin
Connections:
- net VIN: no longer names the net of L1.1
Other:
- note added: "check VIN from boost converter, piezo 12V driving circuit, also i think its accidentally used in PD circuit? on safe pwr fet"
Changed lines of the file:
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@@
+		)
+	)
+	(text "check VIN from boost converter, piezo 12V driving circuit, \nalso i think its accidentally used in PD circuit? \non safe pwr fet"
+		(exclude_from_sim no)
+		(at 143.002 182.372 0)
+		(effects
+			(font
+				(size 1.27 1.27)
+			)
 		)
 	)
@@
 				(hide yes)
 			)
-		)
-	)
-	(global_label "VIN"
-		(shape input)
-		(at 53.34 160.02 90)
-		(fields_autoplaced yes)
-		(effects
-			(font
-				(size 1.27 1.27)
-			)
-			(justify left)
-		)
-		(property "Intersheetrefs" "${INTERSHEET_REFS}"
-			(at 53.34 154.0109 90)
-			(effects
-				(font
-					(size 1.27 1.27)
-				)
-				(justify left)
-				(hide yes)
-			)

Commit message: update after lab session with gustav saturday
Parts:
- removed J3: Haptic Power and GND, Connector_JST:JST_XH_S2B-XH-A_1x02_P2.50mm_Horizontal, symbol Connector:Conn_01x02_Socket
- removed J5: JST CONN from MCU, Connector_JST:JST_XH_S3B-XH-A_1x03_P2.50mm_Horizontal, symbol Connector:Conn_01x03_Socket
- added R53, R54, R55: 3.3k, Resistor_SMD:R_0805_2012Metric_Pad1.20x1.40mm_HandSolder, symbol Device:R
Connections:
- net +3V3: now also R53.1, R54.1, R55.1
- net MCU PWM: now also U2.8 (IO32)
- net PD_INT: now also R53.2
- net SCL: now also R55.2
- net SDA: now also R54.2

Commit message: finished PCB design and gerbers are in directory
Parts:
- removed J15: Conn_01x04_Socket, Connector_JST:JST_XH_S4B-XH-A_1x04_P2.50mm_Horizontal, symbol Connector:Conn_01x04_Socket
- removed JP1, JP2: SolderJumper_2_Open, Jumper:SolderJumper-2_P1.3mm_Open_RoundedPad1.0x1.5mm, symbol Jumper:SolderJumper_2_Open
- removed Q1: NMOS IRLZ44NPBF, Package_TO_SOT_THT:TO-220-3_Horizontal_TabDown, symbol Simulation_SPICE:NMOS
- removed R53: 3.3k, Resistor_SMD:R_0805_2012Metric_Pad1.20x1.40mm_HandSolder, symbol Device:R
- removed S3: 430773034825, EXT_AI_DEPUTY_Library:430773034825, symbol Wurth Buttons:430773034825
- added H1, H2, H3, H4, H5, H6: MountingHole, MountingHole:MountingHole_3mm, symbol Mechanical:MountingHole
- added J12, J7: Conn_01x01_Pin, TestPoint:TestPoint_Pad_4.0x4.0mm, symbol Connector:Conn_01x01_Pin
- added Q3: Q_NMOS_GDS_IRLZ44N, Package_TO_SOT_THT:TO-220-3_Horizontal_TabDown, symbol Transistor_FET_Other:Q_NMOS_Depletion_GDS
- added R5: 3.3k, Resistor_SMD:R_0805_2012Metric_Pad1.20x1.40mm_HandSolder, symbol Device:R
- added S3: L101121MS02Q, EXT_AI_DEPUTY_Library:PWR_SW_L101021MS02Q, symbol PWR_SWITCH:L101121MS02Q
- L1: footprint (none) -> Inductor_SMD:L_Wuerth_WE-PD-Typ-LS
- R47: value 68 -> 100
Connections:
- net +3V3: now also R5.1
- net GND: now also J12.1 (Pin_1), Q3.3 (S)
- net NIRQ: now also R5.2
- net ESPDACOUTL: now reaches U2.10 (IO25)
- net ESPDACOUTR: now reaches U2.11 (IO26)
- net +VDC: now reaches L1.1
- net +VDC: now also S3.2
- net at C1.2, L1.2: now also Q3.2 (D)
- net at R3.1, R47.1: now also Q3.1 (G)
- net MUTE: no longer names the net of U2.37 (IO23)
- net PD_INT: no longer names the net of U2.31 (IO19)
- new net +BATT: J7.1 (Pin_1), S3.1
Other:
- note added: "+Batt Pads for input from BMS"
- note added: "REMEMBER TO ADD Power Button and BL link button POWER BUTTON, due to design change is going to be a slide switch"
- note removed: "REMEMBER TO ADD Power Button and BL link button"

Commit message: updated pcb code
Parts:
- R8: value 10k -> 43
Changed lines of the file:
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@@
 			)
 		)
-		(property "Value" "10k"
+		(property "Value" "43"
 			(at 185.42 54.6099 0)
 			(effects
