File: PCB_Expert_in_Teams/pcb/AI_deputy_PCB/audio_amp.kicad_sch (KiCad schematic)
At the start: 40 parts, among them IC4 IS31AP2005-SLS2-TR, IC5 IS31AP2005-SLS2-TR, IC9 PCM5102APWR, J13 Conn_01x02_Socket, J14 Conn_01x02_Socket, J8 Conn_01x04_Socket

Commit message: finished PCB design and gerbers are in directory
Parts:
- removed J8: Conn_01x04_Socket, Connector_JST:JST_XH_S4B-XH-A-1_1x04_P2.50mm_Horizontal, symbol Connector:Conn_01x04_Socket
- added C61: 4u7, Capacitor_SMD:C_0805_2012Metric_Pad1.18x1.45mm_HandSolder, symbol Device:C
- added JP3, JP4, JP5, JP6: Jumper_3_Open, Jumper:SolderJumper-3_P1.3mm_Open_Pad1.0x1.5mm_NumberLabels, symbol Jumper:Jumper_3_Open
- added R1: 2.7k, Resistor_SMD:R_0805_2012Metric_Pad1.20x1.40mm_HandSolder, symbol Device:R
- IC9: footprint SOP65P640X120-20N -> EXT_AI_DEPUTY_Library:SOP65P640X120-20N
- R41: value 10k -> 7.5k
Connections:
- net +3V3: now also C61.1, JP3.3 (B), JP4.1 (A)
- net GND: now also IC9.12 (SCK), C61.2, JP3.1 (A), JP4.3 (B), R1.1; no longer IC9.11 (FLT), IC9.16 (FMT)
- net Signal Left: now also JP5.2 (C); no longer C57.1, R43.2
- net Signal Right: now also JP6.2 (C); no longer C56.1, R42.2
- net MUTE: no longer names the net of IC9.17 (XSMT), R41.1
- net MUTE: now also R1.2
- new net: IC9.11 (FLT), JP3.2 (C)
- new net: IC9.16 (FMT), JP4.2 (C)
- new net DAC_OUTL: C57.1, JP5.1 (A), R43.2
- new net DAC_OUTR: C56.1, JP6.1 (A), R42.2
- new net ESPDACOUTL: JP5.3 (B)
- new net ESPDACOUTR: JP6.3 (B)
- no-connect marks 1 -> 0
Other:
- note added: "RC delay circuit for soft unmute aka no pops in speakers"
- note added: "i2S should be same trace length Diff. Pairs"
- note removed: "i2S should be same trace length"
- moved on the sheet: R41

Commit message: updated pcb code
Parts:
- removed R1: 2.7k, Resistor_SMD:R_0805_2012Metric_Pad1.20x1.40mm_HandSolder, symbol Device:R
- R41: value 7.5k -> 8.2k
Changed lines of the file:
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@@
 	)
 	(junction
-		(at 120.65 78.74)
-		(diameter 0)
-		(color 0 0 0 0)
-	)
-	(junction
 		(at 36.83 74.93)
 		(diameter 0)
@@
 	)
 	(symbol
-		(lib_id "Device:R")
-		(at 120.65 82.55 0)
-		(mirror x)
-		(unit 1)
-		(exclude_from_sim no)
-		(in_bom yes)
-		(on_board yes)
-		(dnp no)
-		(property "Reference" "R1"
-			(at 116.078 81.28 0)
-			(effects
-				(font
-					(size 1.27 1.27)
-				)
-			)
-		)
-		(property "Value" "2.7k"
-			(at 116.332 83.312 0)
-			(effects
-				(font
-					(size 1.27 1.27)
-				)
-			)
-		)
-		(property "Footprint" "Resistor_SMD:R_0805_2012Metric_Pad1.20x1.40mm_HandSolder"
-			(at 118.872 82.55 90)
-			(effects
-				(font
-					(size 1.27 1.27)
-				)
-				(hide yes)
-			)
-		)
-		(property "Datasheet" "~"
-			(at 120.65 82.55 0)
-			(effects
-				(font
-					(size 1.27 1.27)
-				)
-				(hide yes)
-			)
-		)
-		(property "Description" "Resistor"
-			(at 120.65 82.55 0)
-			(effects
-				(font
-					(size 1.27 1.27)
-				)
-				(hide yes)
-			)
-		)
-		(pin "2"
-		)
-		(pin "1"
-		)
-		(instances
-			(project "AI_deputy_PCB"
-				(path "/3784b751-4d5b-4452-8288-14e483e1cb48/4600983a-86b8-49e8-8db6-b0ddbc3ab361"
-					(reference "R1")
-					(unit 1)
-				)
-			)
-		)
-	)
-	(symbol
 		(lib_id "power:GND")
 		(at 143.51 50.8 270)
@@
 	)
 	(symbol
-		(lib_id "power:GND")
-		(at 120.65 86.36 0)
-		(unit 1)
-		(exclude_from_sim no)
-		(in_bom yes)
-		(on_board yes)
-		(dnp no)
-		(property "Reference" "#PWR020"
-			(at 120.65 92.71 0)
-			(effects
-				(font
-					(size 1.27 1.27)
-				)
-				(hide yes)
-			)
-		)
-		(property "Value" "GND"
-			(at 120.904 90.678 0)
-			(effects
-				(font
-					(size 1.27 1.27)
-				)
-			)
-		)
-		(property "Footprint" ""
-			(at 120.65 86.36 0)
-			(effects
-				(font
-					(size 1.27 1.27)
-				)
-				(hide yes)
-			)
-		)
-		(property "Datasheet" ""
-			(at 120.65 86.36 0)
-			(effects
-				(font
-					(size 1.27 1.27)
-				)
-				(hide yes)
-			)
-		)
-		(property "Description" "Power symbol creates a global label with name \"GND\" , ground"
-			(at 120.65 86.36 0)
-			(effects
-				(font
-					(size 1.27 1.27)
-				)
-				(hide yes)
-			)
-		)
-		(pin "1"
-		)
-		(instances
-			(project "AI_deputy_PCB"
-				(path "/3784b751-4d5b-4452-8288-14e483e1cb48/4600983a-86b8-49e8-8db6-b0ddbc3ab361"
-					(reference "#PWR020")
-					(unit 1)
-				)
-			)
-		)
-	)
-	(symbol
 		(lib_id "power:+3V3")
 		(at 215.9 50.8 270)
@@
 			)
 		)
-		(property "Value" "7.5k"
+		(property "Value" "8.2k"
 			(at 116.332 75.692 0)
 			(effects

Commit message: final push
Other:
- note added: "Had to delete the pull down resistor cause xsmt needs 3.3V"
Changed lines of the file:
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@@
+		)
+	)
+	(text "Had to delete the pull down resistor cause xsmt needs 3.3V \n"
+		(exclude_from_sim no)
+		(at 171.196 78.486 0)
+		(effects
+			(font
+				(size 1.27 1.27)
+			)
 		)
 	)
